File: Production/XRP_Controller-Panel.brd (EAGLE design)
At the start: 147.6 x 177.2 mm, 1332 parts, among them J1 POWER_JACKPOWER_JACK_SLOT, J10 JST_6_PIN_VERTICAL, J11 JST_6_PIN_VERTICAL, J12 Vertical Qwiic Connector, J13 Vertical Qwiic Connector, J14 Vertical Qwiic Connector, J15 JST_6_PIN_VERTICAL, J18 Vertical Qwiic Connector, J19 Vertical Qwiic Connector, J2 JST_6_PIN_VERTICAL, J20 Vertical Qwiic Connector, J21 Vertical Qwiic Connector, J22 POWER_JACKPOWER_JACK_SLOT, J23 JST_6_PIN_VERTICAL, J24 JST_6_PIN_VERTICAL, J25 JST_6_PIN_VERTICAL, J26 JST_6_PIN_VERTICAL, J29 Vertical Qwiic Connector, J3 JST_6_PIN_VERTICAL, J30 Vertical Qwiic Connector, J31 Vertical Qwiic Connector, J32 Vertical Qwiic Connector, J33 POWER_JACKPOWER_JACK_SLOT, J34 JST_6_PIN_VERTICAL, J35 JST_6_PIN_VERTICAL, J36 JST_6_PIN_VERTICAL, J37 JST_6_PIN_VERTICAL, J4 JST_6_PIN_VERTICAL, J40 Vertical Qwiic Connector, J41 Vertical Qwiic Connector, J42 Vertical Qwiic Connector, J43 Vertical Qwiic Connector, J44 POWER_JACKPOWER_JACK_SLOT, J45 JST_6_PIN_VERTICAL, J46 JST_6_PIN_VERTICAL, J47 JST_6_PIN_VERTICAL, J48 JST_6_PIN_VERTICAL, J5 JST_6_PIN_VERTICAL, J51 Vertical Qwiic Connector, J52 Vertical Qwiic Connector, J53 Vertical Qwiic Connector, J54 Vertical Qwiic Connector, J55 POWER_JACKPOWER_JACK_SLOT, J56 JST_6_PIN_VERTICAL, J57 JST_6_PIN_VERTICAL, J58 JST_6_PIN_VERTICAL, J59 JST_6_PIN_VERTICAL, J6 JST_6_PIN_VERTICAL, J62 Vertical Qwiic Connector, J63 Vertical Qwiic Connector, J64 Vertical Qwiic Connector, J65 Vertical Qwiic Connector, J66 POWER_JACKPOWER_JACK_SLOT, J9 Vertical Qwiic Connector, Q12 20V/4.2A/52mΩ/1.4W, Q13 20V/4.2A/52mΩ/1.4W, Q15 20V/4.2A/52mΩ/1.4W, Q16 20V/4.2A/52mΩ/1.4W, Q19 20V/4.2A/52mΩ/1.4W, Q20 20V/4.2A/52mΩ/1.4W, Q22 20V/4.2A/52mΩ/1.4W, Q23 20V/4.2A/52mΩ/1.4W, Q26 20V/4.2A/52mΩ/1.4W, Q27 20V/4.2A/52mΩ/1.4W, Q29 20V/4.2A/52mΩ/1.4W, Q3 20V/4.2A/52mΩ/1.4W, Q30 20V/4.2A/52mΩ/1.4W, Q33 20V/4.2A/52mΩ/1.4W, Q34 20V/4.2A/52mΩ/1.4W, Q36 20V/4.2A/52mΩ/1.4W, Q37 20V/4.2A/52mΩ/1.4W, Q4 20V/4.2A/52mΩ/1.4W, Q40 20V/4.2A/52mΩ/1.4W, Q41 20V/4.2A/52mΩ/1.4W, Q5 20V/4.2A/52mΩ/1.4W, Q6 20V/4.2A/52mΩ/1.4W, Q8 20V/4.2A/52mΩ/1.4W, Q9 20V/4.2A/52mΩ/1.4W, U1 RPI_PICO_W_XRP, U10 RPI_PICO_W_XRP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

Commit message: Update v10 panel files
Parts:
- added U$583: (no value), output:#IO9#0
- added U$584, U$586, U$592, U$594, U$609: (no value), output:#GND#10
- added U$585, U$587, U$593, U$595: (no value), output:#3V3#4
- added U$588: (no value), output:#IO12#0
- added U$589: (no value), output:#IO13#0
- added U$590: (no value), output:#IO27#0
- added U$591: (no value), output:#IO28#0
- added U$596: (no value), output:#IO26#0
- added U$597: (no value), output:#IO22#0
- added U$598: (no value), output:#IO18#0
- added U$599: (no value), output:#IO19#0
- added U$600: (no value), output:#IO20#0
- added U$601: (no value), output:#IO21#0
- added U$602, U$604, U$606: (no value), output:#GND#0
- added U$603, U$605: (no value), output:#3V3#0
- added U$607: (no value), output:#5V#0
- added U$608: (no value), output:#IO16#0
- added U$610: (no value), output:#IO17#0
- added U$611: (no value), output:#5V#18
- added U$612: (no value), output:#I2C#0
- added U$613: (no value), output:ON0
- added U$614: (no value), output:OFF0
- added U$615, U$634: (no value), output:X0
- added U$616, U$635: (no value), output:Y0
- added U$617, U$636: (no value), output:Z0
- added U$618: (no value), output:#IMU_ADR#0
- added U$619: (no value), output:#LINE#0
- added U$620: (no value), output:#MOTOR_L#0
- added U$621: (no value), output:#MOTOR_3#0
- added U$622: (no value), output:#SERVO_1#0
- added U$623: (no value), output:#MOTOR_R#0
- added U$624: (no value), output:#MOTOR_4#0
- added U$625: (no value), output:#SERVO_2#0
- added U$626: (no value), output:#11V_MAX###0
- added U$627: (no value), output:#5V_#0
- added U$628: (no value), output:#GND_#0
- added U$629: (no value), output:#IO16_#0
- added U$630: (no value), output:#_GND#0
- added U$631: (no value), output:#_5V#0
- added U$632: (no value), output:#_IO17#0
- added U$633: (no value), SparkFun-Aesthetics:POLARITY_MARKING_CENTER_POSITIVE#JPG
- added U$637: (no value), output:#EXTRA#0
- added U$638: (no value), output:#VIN_MEAS#0
- added U$639: (no value), output:USER0
- added U$640: (no value), output:#USER_BTN#0
- added U$641: (no value), output:0X6B0
- added U$642: (no value), output:0X6A0
- added U$643: (no value), output:OPEN#0
- added U$644: (no value), output:CLOSED#0
- added U$645: (no value), XRP_LOGOS:XRP_FULL_LOGO
- added U$646: (no value), output:#VUSB#0
- added U$647: (no value), output:IO220
- added U$648: (no value), output:#RANGE#0
- added U$649: (no value), output:#MOT_MODE_R#4#0
- added U$650: (no value), output:#MOT_MODE_L#3#0
- added U$651: (no value), output:SYS0
- added U$652: (no value), output:MOT0
- added U$653: (no value), output:#MOT#0
- added U$654: (no value), output:#SYS#0
- added U$655: (no value), output:#PWR#0
- added U$656: QWIIC_LOGO, XRP_COMPONENTS:QWIIC_INVERTED
- added U$657: (no value), XRP_COMPONENTS:XRP_URL_3MM
- added U$658: (no value), XRP_COMPONENTS:XRP_URL_5MM
- added U$659: (no value), output:#M3##0
- added U$660: (no value), output:#M3##4
- added U$661: (no value), output:#ML##0
- added U$662: (no value), output:#ML##1
- added U$663: (no value), output:#MR##0
- added U$664: (no value), output:#MR##1
- added U$665: (no value), output:#M4##0
- added U$666: (no value), output:#M4##5
- added U$667: (no value), output:100
- added U$668: (no value), output:110
- added U$669: (no value), output:140
- added U$670: (no value), output:150
- added U$671, U$672: (no value), output:MOTOR_IO0
- added U$673, U$677: (no value), output:#EN#0
- added U$674, U$678: (no value), output:#PH#0
- added U$675: (no value), output:#ML#0
- added U$676: (no value), output:#M3#0
- added U$679: (no value), output:#M4#0
- added U$680: (no value), output:#MR#0
- added U$681: (no value), output:20
- added U$682: (no value), output:30
- added U$683: (no value), output:60
- added U$684: (no value), output:70
- U$100: device output:RESET0 -> output:#ML#0
- U$101: device output:#GND#0 -> output:#M3#0
- U$102: device output:#3V3#0 -> output:100
- U$103: device output:#IO0#0 -> output:110
- U$104: device output:#IO1#0 -> output:140
- U$105: device output:#IO5#0 -> output:150
- U$106: device output:#IO4#0 -> output:#MR#0
- U$107: device output:#GND#0 -> output:#M4#0
- U$108: device output:#3V3#0 -> output:20
- U$109: device output:#IO8#0 -> output:30
- U$110: device output:#IO9#0 -> output:60
- U$111: device output:#GND#10 -> output:70
- U$112: device output:#3V3#4 -> output:PWR0
- U$113: device output:#GND#10 -> output:RESET0
- U$114: device output:#3V3#4 -> output:MOTOR_IO0
- U$115: device output:#IO12#0 -> output:MOTOR_IO0
- U$116: device output:#IO13#0 -> output:#EN#0
- U$117: device output:#IO27#0 -> output:#PH#0
- U$118: device output:#IO28#0 -> output:#GND#0
- U$119, U$233: device output:#GND#10 -> output:#3V3#0
- U$120: device output:#3V3#4 -> output:#IO0#0
- U$121: device output:#GND#10 -> output:#IO1#0
- U$122: device output:#3V3#4 -> output:#IO5#0
- U$123: device output:#IO26#0 -> output:#IO4#0
- U$124: device output:#IO22#0 -> output:#GND#0
- U$125: device output:#IO18#0 -> output:#3V3#0
- U$126: device output:#IO19#0 -> output:#IO8#0
- U$127: device output:#IO20#0 -> output:#IO9#0
- U$128: device output:#IO21#0 -> output:#GND#10
- U$129, U$131: device output:#GND#0 -> output:#3V3#4
- U$130: device output:#3V3#0 -> output:#GND#10
- U$132: device output:#3V3#0 -> output:#IO12#0
- U$133: device output:#GND#0 -> output:#IO13#0
- U$134: device output:#5V#0 -> output:#IO27#0
- U$135: device output:#IO16#0 -> output:#IO28#0
- U$137: device output:#IO17#0 -> output:#3V3#4
- U$138: device output:#5V#18 -> output:#GND#10
- U$139: device output:#I2C#0 -> output:#3V3#4
- U$140: device output:ON0 -> output:#IO26#0
- U$141: device output:OFF0 -> output:#IO22#0
- U$142: device output:X0 -> output:#IO18#0
- U$143: device output:Y0 -> output:#IO19#0
- U$144: device output:Z0 -> output:#IO20#0
- U$145: device output:#IMU_ADR#0 -> output:#IO21#0
- U$146: device output:#LINE#0 -> output:#GND#0
- U$147: device output:#MOTOR_L#0 -> output:#3V3#0
- U$148: device output:#MOTOR_3#0 -> output:#GND#0
- U$149: device output:#SERVO_1#0 -> output:#3V3#0
- U$150: device output:#MOTOR_R#0 -> output:#GND#0
- U$151: device output:#MOTOR_4#0 -> output:#5V#0
- U$152: device output:#SERVO_2#0 -> output:#IO16#0
- U$153, U$250: device output:#11V_MAX###0 -> output:#GND#10
- U$154: device output:#5V_#0 -> output:#IO17#0
- U$155: device output:#GND_#0 -> output:#5V#18
- U$156: device output:#IO16_#0 -> output:#I2C#0
- U$157: device output:#_GND#0 -> output:ON0
- U$158: device output:#_5V#0 -> output:OFF0
- U$159: device output:#_IO17#0 -> output:X0
- U$160: device SparkFun-Aesthetics:POLARITY_MARKING_CENTER_POSITIVE#JPG -> output:Y0
- U$161: device output:X0 -> output:Z0
- U$162: device output:Y0 -> output:#IMU_ADR#0
- U$163: device output:Z0 -> output:#LINE#0
- U$164: device output:#EXTRA#0 -> output:#MOTOR_L#0
- U$165: device output:#VIN_MEAS#0 -> output:#MOTOR_3#0
- U$166: device output:USER0 -> output:#SERVO_1#0
- U$167: device output:#USER_BTN#0 -> output:#MOTOR_R#0
- U$168: device output:0X6B0 -> output:#MOTOR_4#0
- U$169: device output:0X6A0 -> output:#SERVO_2#0
- U$170: device output:OPEN#0 -> output:#11V_MAX###0
- U$171: device output:CLOSED#0 -> output:#5V_#0
- U$172: device XRP_LOGOS:XRP_FULL_LOGO -> output:#GND_#0
- U$173: device output:#VUSB#0 -> output:#IO16_#0
- U$174: device XRP_LOGOS:XRP_LOGO -> output:#_GND#0
- U$175: device output:IO220 -> output:#_5V#0
- U$176: device output:#RANGE#0 -> output:#_IO17#0
- U$177: device output:#MOT_MODE_R#4#0 -> SparkFun-Aesthetics:POLARITY_MARKING_CENTER_POSITIVE#JPG
- U$178: device output:#MOT_MODE_L#3#0 -> output:X0
- U$179: device output:SYS0 -> output:Y0
- U$180: device output:MOT0 -> output:Z0
- U$181: device output:#MOT#0 -> output:#EXTRA#0
- U$182: device output:#SYS#0 -> output:#VIN_MEAS#0
- U$183: device output:#PWR#0 -> output:USER0
- U$184: value QWIIC_LOGO -> (none); device XRP_COMPONENTS:QWIIC_INVERTED -> output:#USER_BTN#0
- U$185: device XRP_COMPONENTS:XRP_URL_3MM -> output:0X6B0
- U$186: device XRP_COMPONENTS:XRP_URL_5MM -> output:0X6A0
- U$187: device output:#M3##0 -> output:OPEN#0
- U$188: device output:#M3##4 -> output:CLOSED#0
- U$189: device output:#ML##0 -> XRP_LOGOS:XRP_FULL_LOGO
- U$190: device output:#ML##1 -> output:#VUSB#0
- U$191: device output:#MR##0 -> output:IO220
- U$192: device output:#MR##1 -> output:#RANGE#0
- U$193: device output:#M4##0 -> output:#MOT_MODE_R#4#0
- U$194: device output:#M4##5 -> output:#MOT_MODE_L#3#0
- U$195: device output:#POWER#0 -> output:SYS0
- U$196: device output:PWR0 -> output:MOT0
- U$197: device output:RESET0 -> output:#MOT#0
- U$198: device output:#GND#0 -> output:#SYS#0
- U$199: device output:#3V3#0 -> output:#PWR#0
- U$200: value (none) -> QWIIC_LOGO; device output:#IO0#0 -> XRP_COMPONENTS:QWIIC_INVERTED
- U$201: device output:#IO1#0 -> XRP_COMPONENTS:XRP_URL_3MM
- U$202: device output:#IO5#0 -> XRP_COMPONENTS:XRP_URL_5MM
- U$203: device output:#IO4#0 -> output:#M3##0
- U$204: device output:#GND#0 -> output:#M3##4
- U$205: device output:#3V3#0 -> output:#ML##0
- U$206: device output:#IO8#0 -> output:#ML##1
- U$207: device output:#IO9#0 -> output:#MR##0
- U$208: device output:#GND#10 -> output:#MR##1
- U$209: device output:#3V3#4 -> output:#M4##0
- U$210: device output:#GND#10 -> output:#M4##5
- U$211: device output:#3V3#4 -> output:100
- U$212: device output:#IO12#0 -> output:110
- U$213: device output:#IO13#0 -> output:140
- U$214: device output:#IO27#0 -> output:150
- U$215: device output:#IO28#0 -> output:MOTOR_IO0
- U$216, U$330: device output:#GND#10 -> output:MOTOR_IO0
- U$217: device output:#3V3#4 -> output:#EN#0
- U$218: device output:#GND#10 -> output:#PH#0
- U$219: device output:#3V3#4 -> output:#ML#0
- U$220: device output:#IO26#0 -> output:#M3#0
- U$221: device output:#IO22#0 -> output:#EN#0
- U$222: device output:#IO18#0 -> output:#PH#0
- U$223: device output:#IO19#0 -> output:#M4#0
- U$224: device output:#IO20#0 -> output:#MR#0
- U$225: device output:#IO21#0 -> output:20
- U$226: device output:#GND#0 -> output:30
- U$227: device output:#3V3#0 -> output:60
- U$228: device output:#GND#0 -> output:70
- U$229: device output:#3V3#0 -> output:#POWER#0
- U$230: device output:#GND#0 -> output:PWR0
- U$231: device output:#5V#0 -> output:RESET0
- U$232: device output:#IO16#0 -> output:#GND#0
- U$234: device output:#IO17#0 -> output:#IO0#0
- U$235: device output:#5V#18 -> output:#IO1#0
- U$236: device output:#I2C#0 -> output:#IO5#0
- U$237: device output:ON0 -> output:#IO4#0
- U$238: device output:OFF0 -> output:#GND#0
- U$239: device output:X0 -> output:#3V3#0
- U$240: device output:Y0 -> output:#IO8#0
- U$241: device output:Z0 -> output:#IO9#0
- U$242: device output:#IMU_ADR#0 -> output:#GND#10
- U$243: device output:#LINE#0 -> output:#3V3#4
- U$244: device output:#MOTOR_L#0 -> output:#GND#10
- U$245: device output:#MOTOR_3#0 -> output:#3V3#4
- U$246: device output:#SERVO_1#0 -> output:#IO12#0
- U$247: device output:#MOTOR_R#0 -> output:#IO13#0
- U$248: device output:#MOTOR_4#0 -> output:#IO27#0
- U$249: device output:#SERVO_2#0 -> output:#IO28#0
- U$251: device output:#5V_#0 -> output:#3V3#4
- U$252: device output:#GND_#0 -> output:#GND#10
- U$253: device output:#IO16_#0 -> output:#3V3#4
- U$254: device output:#_GND#0 -> output:#IO26#0
- U$255: device output:#_5V#0 -> output:#IO22#0
- U$256: device output:#_IO17#0 -> output:#IO18#0
- U$257: device SparkFun-Aesthetics:POLARITY_MARKING_CENTER_POSITIVE#JPG -> output:#IO19#0
- U$258: device output:X0 -> output:#IO20#0
- U$259: device output:Y0 -> output:#IO21#0
- U$260: device output:Z0 -> output:#GND#0
- U$261: device output:#EXTRA#0 -> output:#3V3#0
- U$262: device output:#VIN_MEAS#0 -> output:#GND#0
- U$263: device output:USER0 -> output:#3V3#0
- U$264: device output:#USER_BTN#0 -> output:#GND#0
- U$265: device output:0X6B0 -> output:#5V#0
- U$266: device output:0X6A0 -> output:#IO16#0
- U$267, U$364: device output:OPEN#0 -> output:#GND#10
- U$268: device output:CLOSED#0 -> output:#IO17#0
- U$269: device XRP_LOGOS:XRP_FULL_LOGO -> output:#5V#18
- U$270: device output:#VUSB#0 -> output:#I2C#0
- U$271: device XRP_LOGOS:XRP_LOGO -> output:ON0
- U$272: device output:IO220 -> output:OFF0
- U$273: device output:#RANGE#0 -> output:X0
- U$274: device output:#MOT_MODE_R#4#0 -> output:Y0
- U$275: device output:#MOT_MODE_L#3#0 -> output:Z0
- U$276: device output:SYS0 -> output:#IMU_ADR#0
- U$277: device output:MOT0 -> output:#LINE#0
- U$278: device output:#MOT#0 -> output:#MOTOR_L#0
- U$279: device output:#SYS#0 -> output:#MOTOR_3#0
- U$280: device output:#PWR#0 -> output:#SERVO_1#0
- U$281: value QWIIC_LOGO -> (none); device XRP_COMPONENTS:QWIIC_INVERTED -> output:#MOTOR_R#0
- U$282: device XRP_COMPONENTS:XRP_URL_3MM -> output:#MOTOR_4#0
- U$283: device XRP_COMPONENTS:XRP_URL_5MM -> output:#SERVO_2#0
- U$284: device output:#M3##0 -> output:#11V_MAX###0
- U$285: device output:#M3##4 -> output:#5V_#0
- U$286: device output:#ML##0 -> output:#GND_#0
- U$287: device output:#ML##1 -> output:#IO16_#0
- U$288: device output:#MR##0 -> output:#_GND#0
- U$289: device output:#MR##1 -> output:#_5V#0
- U$290: device output:#M4##0 -> output:#_IO17#0
- U$291: device output:#M4##5 -> SparkFun-Aesthetics:POLARITY_MARKING_CENTER_POSITIVE#JPG
- U$292: device output:#POWER#0 -> output:X0
- U$293: device output:PWR0 -> output:Y0
- U$294: device output:RESET0 -> output:Z0
- U$295: device output:#GND#0 -> output:#EXTRA#0
- U$296: device output:#3V3#0 -> output:#VIN_MEAS#0
- U$297: device output:#IO0#0 -> output:USER0
- U$298: device output:#IO1#0 -> output:#USER_BTN#0
- U$299: device output:#IO5#0 -> output:0X6B0
- U$300: device output:#IO4#0 -> output:0X6A0
- U$301: device output:#GND#0 -> output:OPEN#0
- U$302: device output:#3V3#0 -> output:CLOSED#0
- U$303: device output:#IO8#0 -> XRP_LOGOS:XRP_FULL_LOGO
- U$304: device output:#IO9#0 -> output:#VUSB#0
- U$305: device output:#GND#10 -> output:IO220
- U$306: device output:#3V3#4 -> output:#RANGE#0
- U$307: device output:#GND#10 -> output:#MOT_MODE_R#4#0
- U$308: device output:#3V3#4 -> output:#MOT_MODE_L#3#0
- U$309: device output:#IO12#0 -> output:SYS0
- U$310: device output:#IO13#0 -> output:MOT0
- U$311: device output:#IO27#0 -> output:#MOT#0
- U$312: device output:#IO28#0 -> output:#SYS#0
- U$313, U$427: device output:#GND#10 -> output:#PWR#0
- U$314: value (none) -> QWIIC_LOGO; device output:#3V3#4 -> XRP_COMPONENTS:QWIIC_INVERTED
- U$315: device output:#GND#10 -> XRP_COMPONENTS:XRP_URL_3MM
- U$316: device output:#3V3#4 -> XRP_COMPONENTS:XRP_URL_5MM
- U$317: device output:#IO26#0 -> output:#M3##0
- U$318: device output:#IO22#0 -> output:#M3##4
- U$319: device output:#IO18#0 -> output:#ML##0
- U$320: device output:#IO19#0 -> output:#ML##1
- U$321: device output:#IO20#0 -> output:#MR##0
- U$322: device output:#IO21#0 -> output:#MR##1
- U$323: device output:#GND#0 -> output:#M4##0
- U$324: device output:#3V3#0 -> output:#M4##5
- U$325: device output:#GND#0 -> output:100
- U$326: device output:#3V3#0 -> output:110
- U$327: device output:#GND#0 -> output:140
- U$328: device output:#5V#0 -> output:150
- U$329: device output:#IO16#0 -> output:MOTOR_IO0
- U$331: device output:#IO17#0 -> output:#EN#0
- U$332: device output:#5V#18 -> output:#PH#0
- U$333: device output:#I2C#0 -> output:#ML#0
- U$334: device output:ON0 -> output:#M3#0
- U$335: device output:OFF0 -> output:#EN#0
- U$336: device output:X0 -> output:#PH#0
- U$337: device output:Y0 -> output:#M4#0
- U$338: device output:Z0 -> output:#MR#0
- U$339: device output:#IMU_ADR#0 -> output:20
- U$340: device output:#LINE#0 -> output:30
- U$341: device output:#MOTOR_L#0 -> output:60
- U$342: device output:#MOTOR_3#0 -> output:70
- U$343: device output:#SERVO_1#0 -> output:#POWER#0
- U$344: device output:#MOTOR_R#0 -> output:PWR0
- U$345: device output:#MOTOR_4#0 -> output:RESET0
- U$346: device output:#SERVO_2#0 -> output:#GND#0
- U$347: device output:#11V_MAX###0 -> output:#3V3#0
- U$348: device output:#5V_#0 -> output:#IO0#0
- U$349: device output:#GND_#0 -> output:#IO1#0
- U$350: device output:#IO16_#0 -> output:#IO5#0
- U$351: device output:#_GND#0 -> output:#IO4#0
- U$352: device output:#_5V#0 -> output:#GND#0
- U$353: device output:#_IO17#0 -> output:#3V3#0
- U$354: device SparkFun-Aesthetics:POLARITY_MARKING_CENTER_POSITIVE#JPG -> output:#IO8#0
- U$355: device output:X0 -> output:#IO9#0
- U$356: device output:Y0 -> output:#GND#10
- U$357: device output:Z0 -> output:#3V3#4
- U$358: device output:#EXTRA#0 -> output:#GND#10
- U$359: device output:#VIN_MEAS#0 -> output:#3V3#4
- U$360: device output:USER0 -> output:#IO12#0
- U$361: device output:#USER_BTN#0 -> output:#IO13#0
- U$362: device output:0X6B0 -> output:#IO27#0
- U$363: device output:0X6A0 -> output:#IO28#0
- U$365: device output:CLOSED#0 -> output:#3V3#4
- U$366: device XRP_LOGOS:XRP_FULL_LOGO -> output:#GND#10
- U$367: device output:#VUSB#0 -> output:#3V3#4
- U$368: device XRP_LOGOS:XRP_LOGO -> output:#IO26#0
- U$369: device output:IO220 -> output:#IO22#0
- U$37: device output:PWR0 -> output:#PH#0
- U$370: device output:#RANGE#0 -> output:#IO18#0
- U$371: device output:#MOT_MODE_R#4#0 -> output:#IO19#0
- U$372: device output:#MOT_MODE_L#3#0 -> output:#IO20#0
- U$373: device output:SYS0 -> output:#IO21#0
- U$374: device output:MOT0 -> output:#GND#0
- U$375: device output:#MOT#0 -> output:#3V3#0
- U$376: device output:#SYS#0 -> output:#GND#0
- U$377: device output:#PWR#0 -> output:#3V3#0
- U$378: value QWIIC_LOGO -> (none); device XRP_COMPONENTS:QWIIC_INVERTED -> output:#GND#0
- U$379: device XRP_COMPONENTS:XRP_URL_3MM -> output:#5V#0
- U$380: device XRP_COMPONENTS:XRP_URL_5MM -> output:#IO16#0
- U$381, U$478: device output:#M3##0 -> output:#GND#10
- U$382: device output:#M3##4 -> output:#IO17#0
- U$383: device output:#ML##0 -> output:#5V#18
- U$384: device output:#ML##1 -> output:#I2C#0
- U$385: device output:#MR##0 -> output:ON0
- U$386: device output:#MR##1 -> output:OFF0
- U$387: device output:#M4##0 -> output:X0
- U$388: device output:#M4##5 -> output:Y0
- U$389: device output:#POWER#0 -> output:Z0
- U$390: device output:PWR0 -> output:#IMU_ADR#0
- U$391: device output:RESET0 -> output:#LINE#0
- U$392: device output:#GND#0 -> output:#MOTOR_L#0
- U$393: device output:#3V3#0 -> output:#MOTOR_3#0
- U$394: device output:#IO0#0 -> output:#SERVO_1#0
- U$395: device output:#IO1#0 -> output:#MOTOR_R#0
- U$396: device output:#IO5#0 -> output:#MOTOR_4#0
- U$397: device output:#IO4#0 -> output:#SERVO_2#0
- U$398: device output:#GND#0 -> output:#11V_MAX###0
- U$399: device output:#3V3#0 -> output:#5V_#0
- U$400: device output:#IO8#0 -> output:#GND_#0
- U$401: device output:#IO9#0 -> output:#IO16_#0
- U$402: device output:#GND#10 -> output:#_GND#0
- U$403: device output:#3V3#4 -> output:#_5V#0
- U$404: device output:#GND#10 -> output:#_IO17#0
- U$405: device output:#3V3#4 -> SparkFun-Aesthetics:POLARITY_MARKING_CENTER_POSITIVE#JPG
- U$406: device output:#IO12#0 -> output:X0
- U$407: device output:#IO13#0 -> output:Y0
- U$408: device output:#IO27#0 -> output:Z0
- U$409: device output:#IO28#0 -> output:#EXTRA#0
- U$410, U$524: device output:#GND#10 -> output:#VIN_MEAS#0
- U$411: device output:#3V3#4 -> output:USER0
- U$412: device output:#GND#10 -> output:#USER_BTN#0
- U$413: device output:#3V3#4 -> output:0X6B0
- U$414: device output:#IO26#0 -> output:0X6A0
- U$415: device output:#IO22#0 -> output:OPEN#0
- U$416: device output:#IO18#0 -> output:CLOSED#0
- U$417: device output:#IO19#0 -> XRP_LOGOS:XRP_FULL_LOGO
- U$418: device output:#IO20#0 -> output:#VUSB#0
- U$419: device output:#IO21#0 -> output:IO220
- U$420: device output:#GND#0 -> output:#RANGE#0
- U$421: device output:#3V3#0 -> output:#MOT_MODE_R#4#0
- U$422: device output:#GND#0 -> output:#MOT_MODE_L#3#0
- U$423: device output:#3V3#0 -> output:SYS0
- U$424: device output:#GND#0 -> output:MOT0
- U$425: device output:#5V#0 -> output:#MOT#0
- U$426: device output:#IO16#0 -> output:#SYS#0
- U$428: value (none) -> QWIIC_LOGO; device output:#IO17#0 -> XRP_COMPONENTS:QWIIC_INVERTED
- U$429: device output:#5V#18 -> XRP_COMPONENTS:XRP_URL_3MM
- U$430: device output:#I2C#0 -> XRP_COMPONENTS:XRP_URL_5MM
- U$431: device output:ON0 -> output:#M3##0
- U$432: device output:OFF0 -> output:#M3##4
- U$433: device output:X0 -> output:#ML##0
- U$434: device output:Y0 -> output:#ML##1
- U$435: device output:Z0 -> output:#MR##0
- U$436: device output:#IMU_ADR#0 -> output:#MR##1
- U$437: device output:#LINE#0 -> output:#M4##0
- U$438: device output:#MOTOR_L#0 -> output:#M4##5
- U$439: device output:#MOTOR_3#0 -> output:100
- U$440: device output:#SERVO_1#0 -> output:110
- U$441: device output:#MOTOR_R#0 -> output:140
- U$442: device output:#MOTOR_4#0 -> output:150
- U$443: device output:#SERVO_2#0 -> output:MOTOR_IO0
- U$444: device output:#11V_MAX###0 -> output:MOTOR_IO0
- U$445: device output:#5V_#0 -> output:#EN#0
- U$446: device output:#GND_#0 -> output:#PH#0
- U$447: device output:#IO16_#0 -> output:#ML#0
- U$448: device output:#_GND#0 -> output:#M3#0
- U$449: device output:#_5V#0 -> output:#EN#0
- U$450: device output:#_IO17#0 -> output:#PH#0
- U$451: device SparkFun-Aesthetics:POLARITY_MARKING_CENTER_POSITIVE#JPG -> output:#M4#0
- U$452: device output:X0 -> output:#MR#0
- U$453: device output:Y0 -> output:20
- U$454: device output:Z0 -> output:30
- U$455: device output:#EXTRA#0 -> output:60
- U$456: device output:#VIN_MEAS#0 -> output:70
- U$457: device output:USER0 -> output:#POWER#0
- U$458: device output:#USER_BTN#0 -> output:PWR0
- U$459: device output:0X6B0 -> output:RESET0
- U$460: device output:0X6A0 -> output:#GND#0
- U$461: device output:OPEN#0 -> output:#3V3#0
- U$462: device output:CLOSED#0 -> output:#IO0#0
- U$463: device XRP_LOGOS:XRP_FULL_LOGO -> output:#IO1#0
- U$464: device output:#VUSB#0 -> output:#IO5#0
- U$465: device XRP_LOGOS:XRP_LOGO -> output:#IO4#0
- U$466: device output:IO220 -> output:#GND#0
- U$467: device output:#RANGE#0 -> output:#3V3#0
- U$468: device output:#MOT_MODE_R#4#0 -> output:#IO8#0
- U$469: device output:#MOT_MODE_L#3#0 -> output:#IO9#0
- U$470: device output:SYS0 -> output:#GND#10
- U$471: device output:MOT0 -> output:#3V3#4
- U$472: device output:#MOT#0 -> output:#GND#10
- U$473: device output:#SYS#0 -> output:#3V3#4
- U$474: device output:#PWR#0 -> output:#IO12#0
- U$475: value QWIIC_LOGO -> (none); device XRP_COMPONENTS:QWIIC_INVERTED -> output:#IO13#0
- U$476: device XRP_COMPONENTS:XRP_URL_3MM -> output:#IO27#0
- U$477: device XRP_COMPONENTS:XRP_URL_5MM -> output:#IO28#0
- U$479: device output:#M3##4 -> output:#3V3#4
- U$480: device output:#ML##0 -> output:#GND#10
- U$481: device output:#ML##1 -> output:#3V3#4
- U$482: device output:#MR##0 -> output:#IO26#0
- U$483: device output:#MR##1 -> output:#IO22#0
- U$484: device output:#M4##0 -> output:#IO18#0
- U$485: device output:#M4##5 -> output:#IO19#0
- U$486: device output:#POWER#0 -> output:#IO20#0
- U$487: device output:PWR0 -> output:#IO21#0
- U$488: device output:RESET0 -> output:#GND#0
- U$489: device output:#GND#0 -> output:#3V3#0
- U$490: device output:#3V3#0 -> output:#GND#0
- U$491: device output:#IO0#0 -> output:#3V3#0
- U$492: device output:#IO1#0 -> output:#GND#0
- U$493: device output:#IO5#0 -> output:#5V#0
- U$494: device output:#IO4#0 -> output:#IO16#0
- U$495: device output:#GND#0 -> output:#GND#10
- U$496: device output:#3V3#0 -> output:#IO17#0
- U$497: device output:#IO8#0 -> output:#5V#18
- U$498: device output:#IO9#0 -> output:#I2C#0
- U$499: device output:#GND#10 -> output:ON0
- U$500: device output:#3V3#4 -> output:OFF0
- U$501: device output:#GND#10 -> output:X0
- U$502: device output:#3V3#4 -> output:Y0
- U$503: device output:#IO12#0 -> output:Z0
- U$504: device output:#IO13#0 -> output:#IMU_ADR#0
- U$505: device output:#IO27#0 -> output:#LINE#0
- U$506: device output:#IO28#0 -> output:#MOTOR_L#0
- U$507: device output:#GND#10 -> output:#MOTOR_3#0
- U$508: device output:#3V3#4 -> output:#SERVO_1#0
- U$509: device output:#GND#10 -> output:#MOTOR_R#0
- U$510: device output:#3V3#4 -> output:#MOTOR_4#0
- U$511: device output:#IO26#0 -> output:#SERVO_2#0
- U$512: device output:#IO22#0 -> output:#11V_MAX###0
- U$513: device output:#IO18#0 -> output:#5V_#0
- U$514: device output:#IO19#0 -> output:#GND_#0
- U$515: device output:#IO20#0 -> output:#IO16_#0
- U$516: device output:#IO21#0 -> output:#_GND#0
- U$517: device output:#GND#0 -> output:#_5V#0
- U$518: device output:#3V3#0 -> output:#_IO17#0
- U$519: device output:#GND#0 -> SparkFun-Aesthetics:POLARITY_MARKING_CENTER_POSITIVE#JPG
- U$520: device output:#3V3#0 -> output:X0
- U$521: device output:#GND#0 -> output:Y0
- U$522: device output:#5V#0 -> output:Z0
- U$523: device output:#IO16#0 -> output:#EXTRA#0
- U$525: device output:#IO17#0 -> output:USER0
- U$526: device output:#5V#18 -> output:#USER_BTN#0
- U$527: device output:#I2C#0 -> output:0X6B0
- U$528: device output:ON0 -> output:0X6A0
- U$529: device output:OFF0 -> output:OPEN#0
- U$530: device output:X0 -> output:CLOSED#0
- U$531: device output:Y0 -> XRP_LOGOS:XRP_FULL_LOGO
- U$532: device output:Z0 -> output:#VUSB#0
- U$533: device output:#IMU_ADR#0 -> output:IO220
- U$534: device output:#LINE#0 -> output:#RANGE#0
- U$535: device output:#MOTOR_L#0 -> output:#MOT_MODE_R#4#0
- U$536: device output:#MOTOR_3#0 -> output:#MOT_MODE_L#3#0
- U$537: device output:#SERVO_1#0 -> output:SYS0
- U$538: device output:#MOTOR_R#0 -> output:MOT0
- U$539: device output:#MOTOR_4#0 -> output:#MOT#0
- U$540: device output:#SERVO_2#0 -> output:#SYS#0
- U$541: device output:#11V_MAX###0 -> output:#PWR#0
- U$542: value (none) -> QWIIC_LOGO; device output:#5V_#0 -> XRP_COMPONENTS:QWIIC_INVERTED
- U$543: device output:#GND_#0 -> XRP_COMPONENTS:XRP_URL_3MM
- U$544: device output:#IO16_#0 -> XRP_COMPONENTS:XRP_URL_5MM
- U$545: device output:#_GND#0 -> output:#M3##0
- U$546: device output:#_5V#0 -> output:#M3##4
- U$547: device output:#_IO17#0 -> output:#ML##0
- U$548: device SparkFun-Aesthetics:POLARITY_MARKING_CENTER_POSITIVE#JPG -> output:#ML##1
- U$549: device output:X0 -> output:#MR##0
- U$550: device output:Y0 -> output:#MR##1
- U$551: device output:Z0 -> output:#M4##0
- U$552: device output:#EXTRA#0 -> output:#M4##5
- U$553: device output:#VIN_MEAS#0 -> output:100
- U$554: device output:USER0 -> output:110
- U$555: device output:#USER_BTN#0 -> output:140
- U$556: device output:0X6B0 -> output:150
- U$557: device output:0X6A0 -> output:MOTOR_IO0
- U$558: device output:OPEN#0 -> output:MOTOR_IO0
- U$559: device output:CLOSED#0 -> output:#EN#0
- U$560: device XRP_LOGOS:XRP_FULL_LOGO -> output:#PH#0
- U$561: device output:#VUSB#0 -> output:#ML#0
- U$562: device XRP_LOGOS:XRP_LOGO -> output:#M3#0
- U$563: device output:IO220 -> output:#EN#0
- U$564: device output:#RANGE#0 -> output:#PH#0
- U$565: device output:#MOT_MODE_R#4#0 -> output:#M4#0
- U$566: device output:#MOT_MODE_L#3#0 -> output:#MR#0
- U$567: device output:SYS0 -> output:20
- U$568: device output:MOT0 -> output:30
- U$569: device output:#MOT#0 -> output:60
- U$570: device output:#SYS#0 -> output:70
- U$571: device output:#PWR#0 -> output:#POWER#0
- U$572: value QWIIC_LOGO -> (none); device XRP_COMPONENTS:QWIIC_INVERTED -> output:PWR0
- U$573: device XRP_COMPONENTS:XRP_URL_3MM -> output:RESET0
- U$574: device XRP_COMPONENTS:XRP_URL_5MM -> output:#GND#0
- U$575: device output:#M3##0 -> output:#3V3#0
- U$576: device output:#M3##4 -> output:#IO0#0
- U$577: device output:#ML##0 -> output:#IO1#0
- U$578: device output:#ML##1 -> output:#IO5#0
- U$579: device output:#MR##0 -> output:#IO4#0
- U$580: device output:#MR##1 -> output:#GND#0
- U$581: device output:#M4##0 -> output:#3V3#0
- U$582: device output:#M4##5 -> output:#IO8#0
- U$65: device XRP_LOGOS:XRP_LOGO -> output:#EN#0
- moved U$199 142.3 mm to (126.2, 9.53), flipped to the bottom, turned to 90 degrees
- moved U$411 140.6 mm to (116.7, 68.5), turned to 270 degrees
- moved U$397 138.1 mm to (121.5, 73.5), turned to 270 degrees
- moved U$426 137.7 mm to (123.4, 65.3), flipped to the bottom
- moved U$425 137.7 mm to (123.4, 62.7), flipped to the bottom
- moved U$198 137.7 mm to (123.4, 10.8), flipped to the bottom
- moved U$424 137.4 mm to (125.1, 64.0)
- moved U$437 136.3 mm to (123.2, 79.9)
- moved U$197 135.4 mm to (123.4, 8.26), flipped to the bottom
- moved U$408 134.1 mm to (118.0, 78.0), flipped to the bottom, turned to 0 degrees
- moved U$216 132.8 mm to (126.6, 45.1), turned to 270 degrees
- moved U$438 132.6 mm to (123.2, 80.9), turned to 0 degrees
- moved U$396 131.1 mm to (119.3, 82.4), turned to 270 degrees
- moved U$214 126.4 mm to (122.8, 45.7), turned to 270 degrees
- moved U$569 126.3 mm to (3.43, 156.6), flipped to the top, turned to 90 degrees
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Routing:
- net N$40: track 16.8 -> 43.0 mm, vias 1 -> 3
- net N$17: track 16.8 -> 43.0 mm, vias 1 -> 3
- net N$84: track 16.8 -> 43.0 mm, vias 1 -> 3
- net N$62: track 16.8 -> 43.0 mm, vias 1 -> 3
- net N$106: track 16.8 -> 43.0 mm, vias 1 -> 3
- net N$128: track 16.8 -> 43.0 mm, vias 1 -> 3
- net N$83: track 13.0 -> 5.59 mm
- net N$61: track 13.0 -> 5.59 mm
- net N$39: track 13.0 -> 5.59 mm
- net N$12: track 13.0 -> 5.59 mm
- net N$127: track 13.0 -> 5.59 mm
- net N$105: track 13.0 -> 5.59 mm
- net VIN5: track 147.2 -> 150.2 mm
- net VIN4: track 147.2 -> 150.2 mm
- net VIN3: track 147.2 -> 150.2 mm
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